File: 01_top_plate/GL516_Template.kicad_pcb (KiCad board)
At the start: 2 copper layers, 314.4 x 98.8 mm, 90 parts, among them J10 Conn_01x01, J11 Conn_01x01, J12 Conn_01x01, J13 Conn_01x01, J14 Conn_01x01, J15 Conn_01x01, J16 Conn_01x01, J17 Conn_01x01, J2 Conn_01x01, J3 Conn_01x01, J4 Conn_01x01, J5 Conn_01x01, J6 Conn_01x01, J7 Conn_01x01, J8 Conn_01x01, J9 Conn_01x01, SW1 SW_PUSH, SW2 KEY_SWITCH, SW3 SW_PUSH, SW4 KEY_SWITCH, SW4 SW_PUSH, SW5 SW_PUSH, SW7 SW_PUSH, SW8 SW_PUSH

Commit message: Finish Creating Top Plate Project
Parts:
- removed the SW4 at (292.9, 57.1)
- removed the SW4 at (271.5, 66.7)
- removed the SW4 at (233.4, 66.7)
- removed the SW4 at (238.1, 28.6)
- removed the SW4 at (214.3, 66.7)
- removed the SW4 at (161.9, 28.6)
- removed the SW4 at (176.2, 66.7)
- removed the SW4 at (181.0, 28.6)
- removed the SW4 at (200.0, 28.6)
- removed the SW4 at (195.3, 66.7)
- removed the SW4 at (142.9, 28.6)
- removed the SW4 at (38.1, 85.7)
- removed the SW4 at (138.1, 66.7)
- removed the SW4 at (123.8, 28.6)
- removed the SW4 at (157.2, 66.7)
- removed the SW4 at (119.1, 66.7)
- removed the SW4 at (104.8, 28.6)
- removed the SW4 at (100.0, 66.7)
- removed the SW4 at (85.7, 28.6)
- removed the SW4 at (81.0, 66.7)
- removed the SW4 at (66.7, 28.6)
- removed the SW4 at (61.9, 66.7)
- removed the SW4 at (276.2, 28.6)
- removed the SW4 at (47.6, 28.6)
- removed the SW4 at (295.3, 28.6)
- removed the SW4 at (314.3, 66.7)
- removed the SW4 at (314.3, 28.6)
- removed the SW4 at (252.4, 66.7)
- removed the SW4 at (219.1, 28.6)
- removed the SW4 at (257.2, 28.6)
- removed the SW5 at (245.3, 104.8)
- removed the SW5 at (221.5, 104.8)
- removed the SW5 at (178.6, 104.8)
- removed the SW5 at (116.7, 104.8)
- removed the SW7 at (31.0, 104.8)
- removed the SW7 at (73.8, 104.8)
- removed the SW7 at (52.4, 104.8)
- removed the SW8 at (200.0, 104.8)
- removed the SW8 at (266.7, 47.6)
- removed the SW8 at (247.7, 47.6)
- removed the SW8 at (228.6, 47.6)
- removed the SW8 at (238.1, 85.7)
- removed the SW8 at (257.2, 85.7)
- removed the SW8 at (276.2, 85.7)
- removed the SW8 at (190.5, 47.6)
- removed the SW8 at (171.4, 47.6)
- removed the SW8 at (200.0, 85.7)
- removed the SW8 at (219.1, 85.7)
- removed the SW8 at (138.1, 104.8)
- removed the SW8 at (209.6, 47.6)
- removed the SW8 at (181.0, 85.7)
- removed the SW8 at (123.8, 85.7)
- removed the SW8 at (152.4, 47.6)
- removed the SW8 at (142.9, 85.7)
- removed the SW8 at (133.3, 47.6)
- removed the SW8 at (161.9, 85.7)
- removed the SW8 at (114.3, 47.6)
- removed the SW8 at (95.2, 104.8)
- removed the SW8 at (104.8, 85.7)
- removed the SW8 at (157.2, 104.8)
- removed the SW8 at (95.2, 47.6)
- removed the SW8 at (85.7, 85.7)
- removed the SW8 at (76.2, 47.6)
- removed the SW8 at (66.7, 85.7)
- removed the SW8 at (57.1, 47.6)
- removed the SW8 at (295.3, 104.8)
- removed the SW8 at (314.3, 104.8)
- removed the SW8 at (276.2, 104.8)
- removed the SW8 at (295.3, 85.7)
- removed the SW8 at (314.3, 47.6)
- removed the SW8 at (314.3, 85.7)
- added SW10: KEY_SWITCH, kbd_SW_Hole:SW_Hole_1, F.Cu at (85.7, 47.6)
- added SW11: KEY_SWITCH, kbd_SW_Hole:SW_Hole_1, F.Cu at (85.7, 66.6)
- added SW12: KEY_SWITCH, kbd_SW_Hole:SW_Hole_1, F.Cu at (85.7, 85.7)
- added SW13: KEY_SWITCH, kbd_SW_Hole:SW_Hole_1, F.Cu at (104.7, 47.6)
- added SW14: KEY_SWITCH, kbd_SW_Hole:SW_Hole_1, F.Cu at (104.7, 66.6)
- added SW15: KEY_SWITCH, kbd_SW_Hole:SW_Hole_1, F.Cu at (104.7, 85.7)
- added SW16: KEY_SWITCH, kbd_SW_Hole:SW_Hole_1, F.Cu at (104.7, 104.7)
- added SW17: KEY_SWITCH, kbd_SW_Hole:SW_Hole_1, F.Cu at (123.8, 47.6)
- added SW18: KEY_SWITCH, kbd_SW_Hole:SW_Hole_1, F.Cu at (123.8, 66.6)
- added SW19: KEY_SWITCH, kbd_SW_Hole:SW_Hole_1, F.Cu at (123.8, 85.7)
- added SW20: KEY_SWITCH, kbd_SW_Hole:SW_Hole_1, F.Cu at (123.8, 104.7)
- added SW21: KEY_SWITCH, kbd_SW_Hole:SW_Hole_1, F.Cu at (142.8, 104.7)
- added SW22: KEY_SWITCH, kbd_SW_Hole:SW_Hole_1, F.Cu at (200.0, 104.7)
- added SW23: KEY_SWITCH, kbd_SW_Hole:SW_Hole_1, F.Cu at (219.0, 47.6)
- added SW24: KEY_SWITCH, kbd_SW_Hole:SW_Hole_1, F.Cu at (219.0, 66.6)
- added SW25: KEY_SWITCH, kbd_SW_Hole:SW_Hole_1, F.Cu at (219.0, 85.7)
- added SW26: KEY_SWITCH, kbd_SW_Hole:SW_Hole_1, F.Cu at (219.0, 104.7)
- added SW27: KEY_SWITCH, kbd_SW_Hole:SW_Hole_1, F.Cu at (238.1, 47.6)
- added SW28: KEY_SWITCH, kbd_SW_Hole:SW_Hole_1, F.Cu at (238.1, 66.6)
- added SW29: KEY_SWITCH, kbd_SW_Hole:SW_Hole_1, F.Cu at (238.1, 85.7)
- added SW30: KEY_SWITCH, kbd_SW_Hole:SW_Hole_1, F.Cu at (238.1, 104.7)
- added SW31: KEY_SWITCH, kbd_SW_Hole:SW_Hole_1, F.Cu at (257.1, 47.6)
- added SW32: KEY_SWITCH, kbd_SW_Hole:SW_Hole_1, F.Cu at (257.1, 66.6)
- added SW33: KEY_SWITCH, kbd_SW_Hole:SW_Hole_1, F.Cu at (257.1, 85.7)
- added SW34: KEY_SWITCH, kbd_SW_Hole:SW_Hole_1, F.Cu at (276.2, 47.6)
- added SW35: KEY_SWITCH, kbd_SW_Hole:SW_Hole_1, F.Cu at (276.2, 66.6)
- added SW36: KEY_SWITCH, kbd_SW_Hole:SW_Hole_1, F.Cu at (276.2, 85.7)
- added SW37: KEY_SWITCH, kbd_SW_Hole:SW_Hole_1, F.Cu at (295.2, 47.6)
- added SW38: KEY_SWITCH, kbd_SW_Hole:SW_Hole_1, F.Cu at (295.2, 66.6)
- added SW39: KEY_SWITCH, kbd_SW_Hole:SW_Hole_1, F.Cu at (295.2, 85.7)
- added SW4: KEY_SWITCH, kbd_SW_Hole:SW_Hole_1, F.Cu at (47.6, 47.6)
- added SW40: KEY_SWITCH, kbd_SW_Hole:SW_Hole_1, F.Cu at (314.3, 47.6)
- added SW41: KEY_SWITCH, kbd_SW_Hole:SW_Hole_1, F.Cu at (314.3, 66.6)
- added SW42: KEY_SWITCH, kbd_SW_Hole:SW_Hole_1, F.Cu at (314.3, 85.7)
- added SW5: KEY_SWITCH, kbd_SW_Hole:SW_Hole_1, F.Cu at (47.6, 66.6)
- added SW6: KEY_SWITCH, kbd_SW_Hole:SW_Hole_1, F.Cu at (47.6, 85.7)
- added SW7: KEY_SWITCH, kbd_SW_Hole:SW_Hole_1, F.Cu at (66.6, 47.6)
- added SW8: KEY_SWITCH, kbd_SW_Hole:SW_Hole_1, F.Cu at (66.6, 66.6)
- added SW9: KEY_SWITCH, kbd_SW_Hole:SW_Hole_1, F.Cu at (66.6, 85.7)
- SW1: value SW_PUSH -> KEY_SWITCH
- SW2: footprint kbd_SW_Hole:SW_Hole_1.5 -> kbd_SW_Hole:SW_Hole_1
- SW3: value SW_PUSH -> KEY_SWITCH; footprint kbd_SW_Hole:SW_Hole_1.75 -> kbd_SW_Hole:SW_Hole_1
- moved SW3 20.3 mm to (28.5, 85.7)
- moved SW2 19.6 mm to (28.5, 66.6)
- moved SW1 19.0 mm to (28.5, 47.6)
