File: 02_assembly_plate/GL516_Template.kicad_pcb (KiCad board)
At the start: 2 copper layers, 304.4 x 98.8 mm, 87 parts, among them J1 Conn_01x02, SW1 SW_PUSH, SW10 SW_PUSH, SW11 SW_PUSH, SW12 SW_PUSH, SW13 SW_PUSH, SW14 SW_PUSH, SW15 SW_PUSH, SW16 SW_PUSH, SW17 SW_PUSH, SW18 SW_PUSH, SW19 SW_PUSH, SW2 SW_PUSH, SW20 SW_PUSH, SW21 SW_PUSH, SW22 SW_PUSH, SW23 SW_PUSH, SW24 SW_PUSH, SW25 SW_PUSH, SW26 SW_PUSH, SW27 SW_PUSH, SW28 SW_PUSH, SW29 SW_PUSH, SW3 SW_PUSH, SW30 SW_PUSH, SW31 SW_PUSH, SW32 SW_PUSH, SW33 SW_PUSH, SW34 SW_PUSH, SW35 SW_PUSH, SW36 SW_PUSH, SW37 SW_PUSH, SW38 SW_PUSH, SW39 SW_PUSH, SW4 SW_PUSH, SW40 SW_PUSH, SW41 SW_PUSH, SW42 SW_PUSH, SW43 SW_PUSH, SW5 SW_PUSH, SW6 SW_PUSH, SW7 SW_PUSH, SW8 SW_PUSH, SW9 SW_PUSH, U1 BLEMicroPro

Commit message: Finish All Wiring
Routing:
- net Row2: track 24.4 -> 497.7 mm, vias 0 -> 2
- net Row1: track 22.4 -> 468.5 mm, vias 0 -> 2
- net Row0: track 24.5 -> 431.7 mm, vias 0 -> 1
- net Row3: track 12.3 -> 361.2 mm, vias 0 -> 2
- net Col6: track 282.9 -> 316.5 mm
Changed lines of the file:
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@@
     (thickness 1.6)
     (drawings 701)
-    (tracks 302)
+    (tracks 340)
     (zones 0)
     (modules 87)
@@
       (effects (font (size 1 1) (thickness 0.15)))
     )
-    (fp_text user RAW (at -9.8155 14.478 270) (layer B.SilkS)
+    (fp_text user RAW (at -9.8155 14.478 270) (layer B.SilkS) hide
       (effects (font (size 0.75 0.5) (thickness 0.125)) (justify mirror))
     )
@@
       (effects (font (size 0.75 0.5) (thickness 0.125)) (justify mirror))
     )
-    (fp_text user VCC (at -9.8155 6.858 270) (layer B.SilkS)
+    (fp_text user VCC (at -9.8155 6.858 270) (layer B.SilkS) hide
       (effects (font (size 0.75 0.5) (thickness 0.125)) (justify mirror))
     )
@@
   (segment (start 55.195 55.065) (end 55.195 57.1) (width 0.25) (layer B.Cu) (net 2))
   (segment (start 36.145 55.065) (end 36.145 57.1) (width 0.25) (layer B.Cu) (net 2))
+  (segment (start 184.735 57.1) (end 36.145 57.1) (width 0.25) (layer F.Cu) (net 2))
+  (segment (start 199.0725 36.195) (end 199.0725 57.05) (width 0.25) (layer F.Cu) (net 2))
+  (segment (start 201.93 33.3375) (end 199.0725 36.195) (width 0.25) (layer F.Cu) (net 2))
+  (segment (start 294.4131 33.3375) (end 201.93 33.3375) (width 0.25) (layer F.Cu) (net 2))
+  (segment (start 199.0725 57.05) (end 199.1225 57.1) (width 0.25) (layer F.Cu) (net 2))
+  (segment (start 297.257 36.1814) (end 294.4131 33.3375) (width 0.25) (layer F.Cu) (net 2))
+  (segment (start 199.1225 57.1) (end 184.735 57.1) (width 0.25) (layer F.Cu) (net 2))
+  (segment (start 321.895 57.1) (end 199.1225 57.1) (width 0.25) (layer F.Cu) (net 2))
+  (via (at 199.1225 57.1) (size 0.8) (drill 0.4) (layers F.Cu B.Cu) (net 2))
   (segment (start 36.145 68.53) (end 36.145 70.565) (width 0.25) (layer B.Cu) (net 3))
   (segment (start 34.225 61.505) (end 36.195 63.475) (width 0.25) (layer B.Cu) (net 3))
@@
   (segment (start 55.195 74.115) (end 55.195 76.15) (width 0.25) (layer B.Cu) (net 4))
   (segment (start 36.145 74.115) (end 36.145 76.15) (width 0.25) (layer B.Cu) (net 4))
+  (segment (start 36.145 76.15) (end 321.895 76.15) (width 0.25) (layer F.Cu) (net 4))
+  (segment (start 299.797 36.1814) (end 291.2381 27.6225) (width 0.25) (layer F.Cu) (net 4))
+  (segment (start 291.2381 27.6225) (end 195.2625 27.6225) (width 0.25) (layer F.Cu) (net 4))
+  (segment (start 195.2625 27.6225) (end 188.595 34.29) (width 0.25) (layer F.Cu) (net 4))
+  (via (at 188.595 54.2925) (size 0.8) (drill 0.4) (layers F.Cu B.Cu) (net 4))
+  (segment (start 188.595 34.29) (end 188.595 54.2925) (width 0.25) (layer F.Cu) (net 4))
+  (via (at 188.595 76.2) (size 0.8) (drill 0.4) (layers F.Cu B.Cu) (net 4))
+  (segment (start 188.595 54.2925) (end 188.595 76.2) (width 0.25) (layer B.Cu) (net 4))
+  (segment (start 188.595 76.2) (end 187.6425 76.2) (width 0.25) (layer F.Cu) (net 4))
   (segment (start 36.145 87.58) (end 36.145 89.615) (width 0.25) (layer B.Cu) (net 5))
   (segment (start 36.145 82.475) (end 36.145 87.58) (width 0.25) (layer B.Cu) (net 5))
@@
   (segment (start 55.195 93.165) (end 55.195 95.2) (width 0.25) (layer B.Cu) (net 6))
   (segment (start 36.145 93.165) (end 36.145 95.2) (width 0.25) (layer B.Cu) (net 6))
+  (segment (start 182.88 34.29) (end 182.88 53.34) (width 0.25) (layer F.Cu) (net 6))
+  (segment (start 190.5 26.67) (end 182.88 34.29) (width 0.25) (layer F.Cu) (net 6))
+  (segment (start 292.8256 26.67) (end 190.5 26.67) (width 0.25) (layer F.Cu) (net 6))
+  (segment (start 302.337 36.1814) (end 292.8256 26.67) (width 0.25) (layer F.Cu) (net 6))
+  (via (at 182.88 54.2925) (size 0.8) (drill 0.4) (layers F.Cu B.Cu) (net 6))
+  (segment (start 182.88 53.34) (end 182.88 54.2925) (width 0.25) (layer F.Cu) (net 6))
+  (via (at 182.83 95.2) (size 0.8) (drill 0.4) (layers F.Cu B.Cu) (net 6))
+  (segment (start 182.88 95.15) (end 182.83 95.2) (width 0.25) (layer B.Cu) (net 6))
+  (segment (start 182.88 54.2925) (end 182.88 95.15) (width 0.25) (layer B.Cu) (net 6))
+  (segment (start 182.83 95.2) (end 36.145 95.2) (width 0.25) (layer F.Cu) (net 6))
+  (segment (start 321.895 95.2) (end 182.83 95.2) (width 0.25) (layer F.Cu) (net 6))
   (segment (start 55.195 49.48) (end 55.195 51.515) (width 0.25) (layer B.Cu) (net 7))
   (segment (start 55.195 44.375) (end 55.195 49.48) (width 0.25) (layer B.Cu) (net 7))
@@
   (segment (start 112.345 112.215) (end 112.345 114.25) (width 0.25) (layer B.Cu) (net 20))
   (segment (start 304.8136 36.1814) (end 304.877 36.1814) (width 0.25) (layer B.Cu) (net 20))
+  (segment (start 112.345 114.25) (end 245.695 114.25) (width 0.25) (layer F.Cu) (net 20))
+  (segment (start 185.7375 25.7175) (end 177.165 34.29) (width 0.25) (layer F.Cu) (net 20))
+  (segment (start 294.4131 25.7175) (end 185.7375 25.7175) (width 0.25) (layer F.Cu) (net 20))
+  (segment (start 177.165 34.29) (end 177.165 53.34) (width 0.25) (layer F.Cu) (net 20))
+  (segment (start 304.877 36.1814) (end 294.4131 25.7175) (width 0.25) (layer F.Cu) (net 20))
+  (segment (start 177.165 53.34) (end 177.165 54.2925) (width 0.25) (layer F.Cu) (net 20))
+  (via (at 177.165 54.2925) (size 0.8) (drill 0.4) (layers F.Cu B.Cu) (net 20))
+  (via (at 177.165 114.3) (size 0.8) (drill 0.4) (layers F.Cu B.Cu) (net 20))
+  (segment (start 177.165 54.2925) (end 177.165 114.3) (width 0.25) (layer B.Cu) (net 20))
   (segment (start 131.395 49.48) (end 131.395 51.515) (width 0.25) (layer B.Cu) (net 21))
   (segment (start 131.395 44.375) (end 131.395 49.48) (width 0.25) (layer B.Cu) (net 21))
@@
   (segment (start 312.42 39.0525) (end 208.5975 39.0525) (width 0.25) (layer F.Cu) (net 55))
   (via (at 208.5975 39.0525) (size 0.8) (drill 0.4) (layers F.Cu B.Cu) (net 55))
-  (segment (start 135.825 99.629499) (end 135.825 102.145) (width 0.25) (layer B.Cu) (net 55))
-  (segment (start 196.401999 39.0525) (end 135.825 99.629499) (width 0.25) (layer B.Cu) (net 55))
-  (segment (start 208.5975 39.0525) (end 196.401999 39.0525) (width 0.25) (layer B.Cu) (net 55))
   (segment (start 307.275 64.045) (end 305.7525 65.5675) (width 0.25) (layer B.Cu) (net 55))
   (segment (start 305.7525 81.5725) (end 307.275 83.095) (width 0.25) (layer B.Cu) (net 55))
   (segment (start 305.7525 46.5175) (end 305.7525 81.5725) (width 0.25) (layer B.Cu) (net 55))
   (segment (start 307.275 44.995) (end 305.7525 46.5175) (width 0.25) (layer B.Cu) (net 55))
+  (segment (start 135.825 42.2925) (end 135.825 102.145) (width 0.25) (layer B.Cu) (net 55))
+  (segment (start 139.065 39.0525) (end 135.825 42.2925) (width 0.25) (layer B.Cu) (net 55))
+  (segment (start 208.5975 39.0525) (end 139.065 39.0525) (width 0.25) (layer B.Cu) (net 55))
   (segment (start 276.1469 22.86) (end 274.6676 21.3807) (width 0.25) (layer B.Cu) (net 56))
   (segment (start 290.2784 22.86) (end 276.1469 22.86) (width 0.25) (layer B.Cu) (net 56))
