File: 02_assembly_plate/GL516_Template.sch (KiCad schematic (older format))
At the start: 103 parts, among them J1 Conn_01x02, J10 Conn_01x01, J11 Conn_01x01, J12 Conn_01x01, J13 Conn_01x01, J14 Conn_01x01, J15 Conn_01x01, J16 Conn_01x01, J17 Conn_01x01, J2 Conn_01x01, J3 Conn_01x01, J4 Conn_01x01, J5 Conn_01x01, J6 Conn_01x01, J7 Conn_01x01, J8 Conn_01x01, J9 Conn_01x01, SW1 SW_PUSH, SW10 SW_PUSH, SW11 SW_PUSH, SW12 SW_PUSH, SW13 SW_PUSH, SW14 SW_PUSH, SW15 SW_PUSH, SW16 SW_PUSH, SW17 SW_PUSH, SW18 SW_PUSH, SW19 SW_PUSH, SW2 SW_PUSH, SW20 SW_PUSH, SW21 SW_PUSH, SW22 SW_PUSH, SW23 SW_PUSH, SW24 SW_PUSH, SW25 SW_PUSH, SW26 SW_PUSH, SW27 SW_PUSH, SW28 SW_PUSH, SW29 SW_PUSH, SW3 SW_PUSH, SW30 SW_PUSH, SW31 SW_PUSH, SW32 SW_PUSH, SW33 SW_PUSH, SW34 SW_PUSH, SW35 SW_PUSH, SW36 SW_PUSH, SW37 SW_PUSH, SW38 SW_PUSH, SW39 SW_PUSH, SW4 SW_PUSH, SW40 SW_PUSH, SW41 SW_PUSH, SW42 SW_PUSH, SW43 SW_PUSH, SW5 SW_PUSH, SW6 SW_PUSH, SW7 SW_PUSH, SW8 SW_PUSH, SW9 SW_PUSH, U1 BLEMicroPro

Commit message: Something on Kairo-zu updated
Parts:
- J1: footprint kbd_Parts:Battery_XH2.5_GL_Connector -> kbd_Parts:Battery_XH2.5_GL_PCB
Changed lines of the file:
@@
 F 0 "J1" H 13968 875 50  0000 C CNN
 F 1 "Conn_01x02" H 13968 966 50  0000 C CNN
-F 2 "kbd_Parts:Battery_XH2.5_GL_Connector" H 14050 1200 50  0001 C CNN
+F 2 "kbd_Parts:Battery_XH2.5_GL_PCB" H 14050 1200 50  0001 C CNN
 F 3 "~" H 14050 1200 50  0001 C CNN
 	1    14050 1200
